Commit message: Pushing new URDF and porting over exact setup from the lab computer

File: ros2_ws/ur10e.urdf (robot description, URDF)
Before this commit: robot ur10e, 15 links, 14 joints
Links:
- link rail_base_link: geometry collision box size=2.0 0.1 0.05; visual box size=3.0 0.1 0.05
Joints:
- joint linear_rail_joint: axis 0 1 0 -> 1 0 0; limit lower=-1.0 upper=1.0 effort=500 velocity=1.0 -> lower=0.0 upper=3.0 effort=500 velocity=5.0

Commit message: Added the original URDF and reverted some minor changes. + Removed world-rail_base_joint and rail_carriage_link from URDF

File: ros2_ws/ur10e.urdf (robot description, URDF)
Before this commit: robot ur10e, 15 links, 14 joints
Links:
- link rail_base_link: geometry collision box size=3.0 0.1 0.05; visual box size=3.0 0.1 0.05
Joints:
- removed joint world-rail_base_joint

Commit message: Re-added world-rail_base_joint and order kinematic chain accordingly

File: ros2_ws/ur10e.urdf (robot description, URDF)
Before this commit: robot ur10e_robot, 15 links, 13 joints
Joints:
- added joint world-rail_base_joint: type fixed, parent world, child rail_base_link, origin xyz=0 0 0 rpy=0 0 0

Commit message: Add the rig's missing geometry: end walls, the payload, and its tumble
Two kinds of geometry the model lacked.

Collision geometry
- End walls 2 ft beyond each end of the 3 m rail. The switch-end wall
  is 2 ft high, so the arm can reach over it; the far-end wall is full
  height. validator.env_bodies lists every environment body, and both
  the collision check and the clearance measure iterate it.
- The payload, as a `payload` link on the flange in tool0's frame: a
  1 ft, 1 in boom, a 6 x 6 x 18 in body on its tip, and two flat
  6 x 12 x 0.125 in wings flush with the body's top, spanning tool0 x.
  Collision boxes are padded (boom to 1.5 in, body and wings by 2 cm).
  RViz draws it from the same URDF.
- The planner's home screen now carries the home posture over the
  whole 0-3 m rail travel (robot_checks.rail_sweep_clearance), since
  homing and rail-only moves take it there and the end walls make
  clearance depend on the carriage position. The executor's docs no
  longer argue from a model uniform along the rail.

Tumbling-body geometry
- The centre of rotation is the body's geometric centre, 21 in out
  along tool0 z (T_EG, still provisional). The placement point is that
  centre; the flange orbits it.
- The recording is turned as a whole so the boom faces out of the
  mounting wall (target_builder.lab_orientation): the narrowest cone
  holding every recorded boom direction is pointed along the wall's
  outward normal. The legacy placement laid the recording's inertial
  axes on the rail's, and with the wings the payload then hit the wall
  in a third of the packaged recording whatever the arm did. Turned,
  it stays at least 397 mm clear with the centre at 0.5 m.

Consequences
- Home is now [0, -75, 100, -115, 100, 90] deg. The old one pointed the
  boom into the mounting wall; wrist 3 at 90 lays the wings across the
  rail, so homing does not swing one into the switch-end wall.
- plans/payload_20261010: a 60 s section (samples 1099-1700) certified
  against all of this; the old wall-mount plan's mount is refused.
  Re-checked by sampling: no collisions at 200 Hz, the centre held to
  within 0.004 mm, payload at least 17 mm from the arm's own links.
- Tests: new ones pin the walls, the payload, the rail sweep and the
  lab orientation. Regressions recorded on a bare flange, and algorithm
  tests built on a posture that puts the payload into the floor, now
  run on a bare-flange copy of the URDF. A failed rclpy.init in the
  executor tests no longer cascades into every later ROS test.

Not covered: the rail sweep stops at 0 m, while the rig homes to
-0.05 m. This home keeps 148 mm there, but the sweep should include it.

594 tests pass in the pinned image (run_tests.sh).

File: ros2_ws/ur10e.urdf (robot description, URDF)
Before this commit: robot ur10e_robot, 15 links, 14 joints
Links:
- added link payload; collision box size=0.0381 0.0381 0.3048; collision box size=0.1924 0.1924 0.4972
Joints:
- added joint flange-payload: type fixed, parent flange, child payload, origin xyz=0 0 0 rpy=1.5707963267948966 0 1.5707963267948966
